File: Hardware/Qwiic_Grideye.brd (EAGLE design)
At the start: 25.4 x 25.4 mm, 26 parts, among them J2 SMD, J3 PTH, J4 SMD, U2 GRIDEYE

Commit message: checklist changes
Routing:
- net 3.3V: track 53.5 -> 58.2 mm
- net SCL: track 58.1 -> 59.2 mm
Other:
- board text added: "ADDR Open-0x3B Close-0x3A"
- board text added: "GridEYE 8x8 IR Array"
- board text added: "I2C PU"
- board text added: "Units in Inches"
- board text removed: "I2C"

Commit message: updated i2c address
Other:
- board text added: "ADDR Open-0x69 Close-0x68"
- board text removed: "ADDR Open-0x3B Close-0x3A"
Changed lines of the file:
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@@
 <text x="7.62" y="2.54" size="1.016" layer="21" font="vector" ratio="15" rot="R90" align="center-left">GND</text>
 <text x="22.86" y="6.477" size="1.016" layer="22" font="vector" ratio="15" rot="MR0">ADDR
-Open-0x3B
-Close-0x3A</text>
+Open-0x69
+Close-0x68</text>
 <text x="10.16" y="2.54" size="1.016" layer="22" font="vector" ratio="15" rot="MR90" align="center-left">3.3V</text>
 <text x="12.7" y="2.54" size="1.016" layer="22" font="vector" ratio="15" rot="MR90" align="center-left">SDA</text>

Commit message: post checklist changes
Other:
- board text added: "v10"
- board text removed: "v01"
Changed lines of the file:
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@@
 <layer number="20" name="Dimension" color="15" fill="1" visible="yes" active="yes"/>
 <layer number="21" name="tPlace" color="16" fill="1" visible="yes" active="yes"/>
-<layer number="22" name="bPlace" color="14" fill="1" visible="yes" active="yes"/>
+<layer number="22" name="bPlace" color="14" fill="1" visible="no" active="yes"/>
 <layer number="23" name="tOrigins" color="15" fill="1" visible="yes" active="yes"/>
 <layer number="24" name="bOrigins" color="15" fill="1" visible="no" active="yes"/>
@@
 <layer number="29" name="tStop" color="7" fill="3" visible="no" active="yes"/>
 <layer number="30" name="bStop" color="7" fill="6" visible="no" active="yes"/>
-<layer number="31" name="tCream" color="7" fill="4" visible="yes" active="yes"/>
-<layer number="32" name="bCream" color="7" fill="5" visible="yes" active="yes"/>
+<layer number="31" name="tCream" color="7" fill="4" visible="no" active="yes"/>
+<layer number="32" name="bCream" color="7" fill="5" visible="no" active="yes"/>
 <layer number="33" name="tFinish" color="6" fill="3" visible="no" active="yes"/>
 <layer number="34" name="bFinish" color="6" fill="6" visible="no" active="yes"/>
@@
 <text x="7.62" y="2.54" size="1.016" layer="22" font="vector" ratio="15" rot="MR90" align="center-left">GND</text>
 <text x="12.7" y="7.112" size="1.016" layer="21" font="vector" ratio="15" rot="SR0" align="center">GridEYE</text>
-<text x="2.413" y="1.27" size="1.27" layer="16" font="vector" ratio="15" rot="MR0" align="center">v01</text>
+<text x="2.413" y="1.27" size="1.27" layer="16" font="vector" ratio="15" rot="MR0" align="center">v10</text>
 <dimension x1="2.54" y1="22.86" x2="22.86" y2="22.86" x3="12.7" y3="31.75" textsize="1.27" textratio="15" layer="47" unit="inch"/>
 <dimension x1="0" y1="25.4" x2="0" y2="0" x3="-8.89" y3="12.7" textsize="1.27" textratio="15" layer="47" unit="inch"/>
