File: Production/Qwiic_Grideye-Panel_v10.brd (EAGLE design)
At the start: 25.4 x 25.4 mm, 24 parts, among them J2 SMD, J3 PTH, J4 SMD, U2 GRIDEYE

Commit message: created panel v10
Parts:
- added C10, C102, C106, C110, C114, C118, C122, C126, C130, C134, C138, C14, C142, C146, C150, C154, C158, C162, C166, C170, C174, C178, C18, C182, C186, C190, C194, C198, C22, C26, C30, C34, C38, C42, C46, C50, C54, C58, C6, C62, C66, C70, C74, C78, C82, C86, C90, C94, C98: 1.0uF, SparkFun-Capacitors:0603
- added C100, C104, C108, C112, C116, C12, C120, C124, C128, C132, C136, C140, C144, C148, C152, C156, C16, C160, C164, C168, C172, C176, C180, C184, C188, C192, C196, C20, C200, C24, C28, C32, C36, C40, C44, C48, C52, C56, C60, C64, C68, C72, C76, C8, C80, C84, C88, C92, C96: 10uF, SparkFun-Capacitors:0603
- added C101, C105, C109, C113, C117, C121, C125, C129, C13, C133, C137, C141, C145, C149, C153, C157, C161, C165, C169, C17, C173, C177, C181, C185, C189, C193, C197, C21, C25, C29, C33, C37, C41, C45, C49, C5, C53, C57, C61, C65, C69, C73, C77, C81, C85, C89, C9, C93, C97: 0.1uF, SparkFun-Capacitors:0603
- added C103, C107, C11, C111, C115, C119, C123, C127, C131, C135, C139, C143, C147, C15, C151, C155, C159, C163, C167, C171, C175, C179, C183, C187, C19, C191, C195, C199, C23, C27, C31, C35, C39, C43, C47, C51, C55, C59, C63, C67, C7, C71, C75, C79, C83, C87, C91, C95, C99: 2.2uF, SparkFun-Capacitors:0603
- added E$1: (no value), SparkFun-Retired:FIDUCIAL-1.5X3
- added E$5, E$8: (no value), SparkFun-Aesthetics:FIDUCIAL-1X2
- added J10, J102, J106, J110, J114, J118, J122, J126, J130, J134, J138, J14, J142, J146, J150, J154, J158, J162, J166, J170, J174, J178, J18, J182, J186, J190, J194, J198, J22, J26, J30, J34, J38, J42, J46, J50, J54, J58, J6, J62, J66, J70, J74, J78, J82, J86, J90, J94, J98: PTH, SparkX:1X04_NO_SILK
- added J100, J104, J108, J112, J116, J12, J120, J124, J128, J132, J136, J140, J144, J148, J152, J156, J16, J160, J164, J168, J172, J176, J180, J184, J188, J192, J196, J20, J200, J24, J28, J32, J36, J40, J44, J48, J52, J56, J60, J64, J68, J72, J76, J8, J80, J84, J88, J92, J96: (no value), SparkFun-Connectors:1X01_NO_SILK
- added J101, J103, J105, J107, J109, J11, J111, J113, J115, J117, J119, J121, J123, J125, J127, J129, J13, J131, J133, J135, J137, J139, J141, J143, J145, J147, J149, J15, J151, J153, J155, J157, J159, J161, J163, J165, J167, J169, J17, J171, J173, J175, J177, J179, J181, J183, J185, J187, J189, J19, J191, J193, J195, J197, J199, J21, J23, J25, J27, J29, J31, J33, J35, J37, J39, J41, J43, J45, J47, J49, J5, J51, J53, J55, J57, J59, J61, J63, J65, J67, J69, J7, J71, J73, J75, J77, J79, J81, J83, J85, J87, J89, J9, J91, J93, J95, J97, J99: SMD, SparkX:1X04_1MM_RA
- added JP10, JP101, JP102, JP104, JP105, JP108, JP109, JP11, JP111, JP112, JP115, JP116, JP118, JP119, JP122, JP123, JP125, JP126, JP129, JP13, JP130, JP132, JP133, JP136, JP137, JP139, JP14, JP140, JP143, JP144, JP146, JP147, JP150, JP151, JP153, JP154, JP157, JP158, JP160, JP161, JP164, JP165, JP167, JP168, JP17, JP171, JP172, JP174, JP175, JP178, JP179, JP18, JP181, JP182, JP185, JP186, JP188, JP189, JP192, JP193, JP195, JP196, JP199, JP20, JP200, JP202, JP203, JP206, JP207, JP209, JP21, JP210, JP213, JP214, JP216, JP217, JP220, JP221, JP223, JP224, JP227, JP228, JP230, JP231, JP234, JP235, JP237, JP238, JP24, JP241, JP242, JP244, JP245, JP248, JP249, JP25, JP251, JP252, JP255, JP256, JP258, JP259, JP262, JP263, JP265, JP266, JP269, JP27, JP270, JP272, JP273, JP276, JP277, JP279, JP28, JP280, JP283, JP284, JP286, JP287, JP290, JP291, JP293, JP294, JP297, JP298, JP300, JP301, JP304, JP305, JP307, JP308, JP31, JP311, JP312, JP314, JP315, JP318, JP319, JP32, JP321, JP322, JP325, JP326, JP328, JP329, JP332, JP333, JP335, JP336, JP339, JP34, JP340, JP342, JP343, JP346, JP347, JP349, JP35, JP350, JP38, JP39, JP41, JP42, JP45, JP46, JP48, JP49, JP52, JP53, JP55, JP56, JP59, JP60, JP62, JP63, JP66, JP67, JP69, JP70, JP73, JP74, JP76, JP77, JP80, JP81, JP83, JP84, JP87, JP88, JP90, JP91, JP94, JP95, JP97, JP98: FIDUCIALUFIDUCIAL, SparkFun:MICRO-FIDUCIAL
- added JP100, JP106, JP107, JP113, JP114, JP120, JP121, JP127, JP128, JP134, JP135, JP141, JP142, JP148, JP149, JP15, JP155, JP156, JP16, JP162, JP163, JP169, JP170, JP176, JP177, JP183, JP184, JP190, JP191, JP197, JP198, JP204, JP205, JP211, JP212, JP218, JP219, JP22, JP225, JP226, JP23, JP232, JP233, JP239, JP240, JP246, JP247, JP253, JP254, JP260, JP261, JP267, JP268, JP274, JP275, JP281, JP282, JP288, JP289, JP29, JP295, JP296, JP30, JP302, JP303, JP309, JP310, JP316, JP317, JP323, JP324, JP330, JP331, JP337, JP338, JP344, JP345, JP36, JP37, JP43, JP44, JP50, JP51, JP57, JP58, JP64, JP65, JP71, JP72, JP78, JP79, JP8, JP85, JP86, JP9, JP92, JP93, JP99: STAND-OFF, SparkFun:STAND-OFF
- added JP103, JP110, JP117, JP12, JP124, JP131, JP138, JP145, JP152, JP159, JP166, JP173, JP180, JP187, JP19, JP194, JP201, JP208, JP215, JP222, JP229, JP236, JP243, JP250, JP257, JP26, JP264, JP271, JP278, JP285, JP292, JP299, JP306, JP313, JP320, JP327, JP33, JP334, JP341, JP348, JP40, JP47, JP54, JP61, JP68, JP75, JP82, JP89, JP96: (no value), SparkFun-Jumpers:SMT-JUMPER_3_2-NC_PASTE_SILK
- added LOGO10, LOGO11, LOGO12, LOGO13, LOGO14, LOGO15, LOGO16, LOGO17, LOGO18, LOGO19, LOGO2, LOGO20, LOGO21, LOGO22, LOGO23, LOGO24, LOGO25, LOGO26, LOGO27, LOGO28, LOGO29, LOGO3, LOGO30, LOGO31, LOGO32, LOGO33, LOGO34, LOGO35, LOGO36, LOGO37, LOGO38, LOGO39, LOGO4, LOGO40, LOGO41, LOGO42, LOGO43, LOGO44, LOGO45, LOGO46, LOGO47, LOGO48, LOGO49, LOGO5, LOGO50, LOGO6, LOGO7, LOGO8, LOGO9: OSHW-LOGOMINI, SparkFun-Aesthetics:OSHW-LOGO-MINI
- added R10, R101, R102, R105, R106, R109, R110, R113, R114, R117, R118, R121, R122, R125, R126, R129, R13, R130, R133, R134, R137, R138, R14, R141, R142, R145, R146, R149, R150, R153, R154, R157, R158, R161, R162, R165, R166, R169, R17, R170, R173, R174, R177, R178, R18, R181, R182, R185, R186, R189, R190, R193, R194, R197, R198, R21, R22, R25, R26, R29, R3, R30, R33, R34, R37, R38, R41, R42, R45, R46, R49, R50, R53, R54, R57, R58, R6, R61, R62, R65, R66, R69, R70, R73, R74, R77, R78, R81, R82, R85, R86, R89, R9, R90, R93, R94, R97, R98: 4.7k, SparkFun-Resistors:0603
- added R100, R104, R108, R112, R116, R12, R120, R124, R128, R132, R136, R140, R144, R148, R152, R156, R16, R160, R164, R168, R172, R176, R180, R184, R188, R192, R196, R20, R200, R24, R28, R32, R36, R40, R44, R48, R52, R56, R60, R64, R68, R72, R76, R8, R80, R84, R88, R92, R96: 20, SparkFun-Resistors:0603
- added R103, R107, R11, R111, R115, R119, R123, R127, R131, R135, R139, R143, R147, R15, R151, R155, R159, R163, R167, R171, R175, R179, R183, R187, R19, R191, R195, R199, R23, R27, R31, R35, R39, R43, R47, R51, R55, R59, R63, R67, R7, R71, R75, R79, R83, R87, R91, R95, R99: 10k, SparkFun-Resistors:0603
- added SJ10, SJ11, SJ12, SJ13, SJ14, SJ15, SJ16, SJ17, SJ18, SJ19, SJ2, SJ20, SJ21, SJ22, SJ23, SJ24, SJ25, SJ26, SJ27, SJ28, SJ29, SJ3, SJ30, SJ31, SJ32, SJ33, SJ34, SJ35, SJ36, SJ37, SJ38, SJ39, SJ4, SJ40, SJ41, SJ42, SJ43, SJ44, SJ45, SJ46, SJ47, SJ48, SJ49, SJ5, SJ50, SJ6, SJ7, SJ8, SJ9: (no value), SparkFun:SJ_2S-NO
- added U$10, U$100, U$12, U$14, U$16, U$18, U$20, U$22, U$24, U$26, U$28, U$30, U$32, U$34, U$36, U$38, U$4, U$40, U$42, U$44, U$46, U$48, U$50, U$52, U$54, U$56, U$58, U$6, U$60, U$62, U$64, U$66, U$68, U$70, U$72, U$74, U$76, U$78, U$8, U$80, U$82, U$84, U$86, U$88, U$90, U$92, U$94, U$96, U$98: SFE_LOGO_NAME.1_INCH, SparkFun-Aesthetics:SFE_LOGO_NAME_.1
- added U$11, U$13, U$15, U$17, U$19, U$21, U$23, U$25, U$27, U$29, U$3, U$31, U$33, U$35, U$37, U$39, U$41, U$43, U$45, U$47, U$49, U$5, U$51, U$53, U$55, U$57, U$59, U$61, U$63, U$65, U$67, U$69, U$7, U$71, U$73, U$75, U$77, U$79, U$81, U$83, U$85, U$87, U$89, U$9, U$91, U$93, U$95, U$97, U$99: SFE_LOGO_NAME_FLAME.1_INCH, SparkFun-Aesthetics:SFE_LOGO_NAME_FLAME_.1
- added U1, U10, U11, U12, U13, U14, U15, U16, U17, U18, U19, U20, U21, U22, U23, U24, U25, U26, U27, U28, U29, U3, U30, U31, U32, U33, U34, U35, U36, U37, U38, U39, U4, U40, U41, U42, U43, U44, U45, U46, U47, U48, U49, U5, U50, U6, U7, U8, U9: GRIDEYE, SparkFun-Sensors:GRIDEYE-AMG88
- moved C2 9.70 mm to (17.0, 25.9)
- moved C3 9.70 mm to (13.2, 25.9)
- moved J1 9.70 mm to (24.6, 8.13)
- moved J2 9.70 mm to (11.9, 19.6)
- moved J4 9.70 mm to (27.2, 19.6)
- moved JP4 9.70 mm to (29.7, 29.7)
- moved JP7 9.70 mm to (19.6, 28.4)
- moved R1 9.70 mm to (25.9, 25.9)
- moved R2 9.70 mm to (24.6, 13.2)
- moved SJ1 9.70 mm to (28.4, 11.9)
- moved U$1 9.70 mm to (13.6, 28.6)
- moved U2 9.70 mm to (19.6, 19.6)
- moved C1 9.70 mm to (22.1, 25.9)
- moved C4 9.70 mm to (14.5, 13.2)
- moved J3 9.70 mm to (14.5, 8.13)
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Connections:
- new net 3.3V1: C5.1, C8.1, J5.2, J6.2, J7.2, JP12.2, R7.2, U1.13, U1.9
- new net 3.3V10: C41.1, C44.1, J41.2, J42.2, J43.2, JP75.2, R43.2, U11.13, U11.9
- new net 3.3V11: C45.1, C48.1, J45.2, J46.2, J47.2, JP82.2, R47.2, U12.13, U12.9
- new net 3.3V12: C49.1, C52.1, J49.2, J50.2, J51.2, JP89.2, R51.2, U13.13, U13.9
- new net 3.3V13: C53.1, C56.1, J53.2, J54.2, J55.2, JP96.2, R55.2, U14.13, U14.9
- new net 3.3V14: C57.1, C60.1, J57.2, J58.2, J59.2, JP103.2, R59.2, U15.13, U15.9
- new net 3.3V15: C61.1, C64.1, J61.2, J62.2, J63.2, JP110.2, R63.2, U16.13, U16.9
- new net 3.3V16: C65.1, C68.1, J65.2, J66.2, J67.2, JP117.2, R67.2, U17.13, U17.9
- new net 3.3V17: C69.1, C72.1, J69.2, J70.2, J71.2, JP124.2, R71.2, U18.13, U18.9
- new net 3.3V18: C73.1, C76.1, J73.2, J74.2, J75.2, JP131.2, R75.2, U19.13, U19.9
- new net 3.3V19: C77.1, C80.1, J77.2, J78.2, J79.2, JP138.2, R79.2, U20.13, U20.9
- new net 3.3V2: C12.1, C9.1, J10.2, J11.2, J9.2, JP19.2, R11.2, U3.13, U3.9
- new net 3.3V20: C81.1, C84.1, J81.2, J82.2, J83.2, JP145.2, R83.2, U21.13, U21.9
- new net 3.3V21: C85.1, C88.1, J85.2, J86.2, J87.2, JP152.2, R87.2, U22.13, U22.9
- new net 3.3V22: C89.1, C92.1, J89.2, J90.2, J91.2, JP159.2, R91.2, U23.13, U23.9
- new net 3.3V23: C93.1, C96.1, J93.2, J94.2, J95.2, JP166.2, R95.2, U24.13, U24.9
- new net 3.3V24: C100.1, C97.1, J97.2, J98.2, J99.2, JP173.2, R99.2, U25.13, U25.9
- new net 3.3V25: C101.1, C104.1, J101.2, J102.2, J103.2, JP180.2, R103.2, U26.13, U26.9
- new net 3.3V26: C105.1, C108.1, J105.2, J106.2, J107.2, JP187.2, R107.2, U27.13, U27.9
- new net 3.3V27: C109.1, C112.1, J109.2, J110.2, J111.2, JP194.2, R111.2, U28.13, U28.9
- new net 3.3V28: C113.1, C116.1, J113.2, J114.2, J115.2, JP201.2, R115.2, U29.13, U29.9
- new net 3.3V29: C117.1, C120.1, J117.2, J118.2, J119.2, JP208.2, R119.2, U30.13, U30.9
- new net 3.3V3: C13.1, C16.1, J13.2, J14.2, J15.2, JP26.2, R15.2, U4.13, U4.9
- new net 3.3V30: C121.1, C124.1, J121.2, J122.2, J123.2, JP215.2, R123.2, U31.13, U31.9
- new net 3.3V31: C125.1, C128.1, J125.2, J126.2, J127.2, JP222.2, R127.2, U32.13, U32.9
- new net 3.3V32: C129.1, C132.1, J129.2, J130.2, J131.2, JP229.2, R131.2, U33.13, U33.9
- new net 3.3V33: C133.1, C136.1, J133.2, J134.2, J135.2, JP236.2, R135.2, U34.13, U34.9
- new net 3.3V34: C137.1, C140.1, J137.2, J138.2, J139.2, JP243.2, R139.2, U35.13, U35.9
- new net 3.3V35: C141.1, C144.1, J141.2, J142.2, J143.2, JP250.2, R143.2, U36.13, U36.9
- new net 3.3V36: C145.1, C148.1, J145.2, J146.2, J147.2, JP257.2, R147.2, U37.13, U37.9
- new net 3.3V37: C149.1, C152.1, J149.2, J150.2, J151.2, JP264.2, R151.2, U38.13, U38.9
- new net 3.3V38: C153.1, C156.1, J153.2, J154.2, J155.2, JP271.2, R155.2, U39.13, U39.9
- new net 3.3V39: C157.1, C160.1, J157.2, J158.2, J159.2, JP278.2, R159.2, U40.13, U40.9
- new net 3.3V4: C17.1, C20.1, J17.2, J18.2, J19.2, JP33.2, R19.2, U5.13, U5.9
- new net 3.3V40: C161.1, C164.1, J161.2, J162.2, J163.2, JP285.2, R163.2, U41.13, U41.9
- new net 3.3V41: C165.1, C168.1, J165.2, J166.2, J167.2, JP292.2, R167.2, U42.13, U42.9
- new net 3.3V42: C169.1, C172.1, J169.2, J170.2, J171.2, JP299.2, R171.2, U43.13, U43.9
- new net 3.3V43: C173.1, C176.1, J173.2, J174.2, J175.2, JP306.2, R175.2, U44.13, U44.9
- new net 3.3V44: C177.1, C180.1, J177.2, J178.2, J179.2, JP313.2, R179.2, U45.13, U45.9
- new net 3.3V45: C181.1, C184.1, J181.2, J182.2, J183.2, JP320.2, R183.2, U46.13, U46.9
- new net 3.3V46: C185.1, C188.1, J185.2, J186.2, J187.2, JP327.2, R187.2, U47.13, U47.9
- new net 3.3V47: C189.1, C192.1, J189.2, J190.2, J191.2, JP334.2, R191.2, U48.13, U48.9
- new net 3.3V48: C193.1, C196.1, J193.2, J194.2, J195.2, JP341.2, R195.2, U49.13, U49.9
- new net 3.3V49: C197.1, C200.1, J197.2, J198.2, J199.2, JP348.2, R199.2, U50.13, U50.9
- new net 3.3V5: C21.1, C24.1, J21.2, J22.2, J23.2, JP40.2, R23.2, U6.13, U6.9
- new net 3.3V6: C25.1, C28.1, J25.2, J26.2, J27.2, JP47.2, R27.2, U7.13, U7.9
- new net 3.3V7: C29.1, C32.1, J29.2, J30.2, J31.2, JP54.2, R31.2, U8.13, U8.9
- new net 3.3V8: C33.1, C36.1, J33.2, J34.2, J35.2, JP61.2, R35.2, U9.13, U9.9
- new net 3.3V9: C37.1, C40.1, J37.2, J38.2, J39.2, JP68.2, R39.2, U10.13, U10.9
- new net ADDR1: R7.1, SJ2.2, U1.5
- new net ADDR10: R43.1, SJ11.2, U11.5
- new net ADDR11: R47.1, SJ12.2, U12.5
- new net ADDR12: R51.1, SJ13.2, U13.5
- new net ADDR13: R55.1, SJ14.2, U14.5
- new net ADDR14: R59.1, SJ15.2, U15.5
- new net ADDR15: R63.1, SJ16.2, U16.5
- new net ADDR16: R67.1, SJ17.2, U17.5
- new net ADDR17: R71.1, SJ18.2, U18.5
- new net ADDR18: R75.1, SJ19.2, U19.5
- new net ADDR19: R79.1, SJ20.2, U20.5
- new net ADDR2: R11.1, SJ3.2, U3.5
- new net ADDR20: R83.1, SJ21.2, U21.5
- new net ADDR21: R87.1, SJ22.2, U22.5
- new net ADDR22: R91.1, SJ23.2, U23.5
- new net ADDR23: R95.1, SJ24.2, U24.5
- new net ADDR24: R99.1, SJ25.2, U25.5
- new net ADDR25: R103.1, SJ26.2, U26.5
- new net ADDR26: R107.1, SJ27.2, U27.5
- new net ADDR27: R111.1, SJ28.2, U28.5
- new net ADDR28: R115.1, SJ29.2, U29.5
- new net ADDR29: R119.1, SJ30.2, U30.5
- new net ADDR3: R15.1, SJ4.2, U4.5
- new net ADDR30: R123.1, SJ31.2, U31.5
- new net ADDR31: R127.1, SJ32.2, U32.5
- new net ADDR32: R131.1, SJ33.2, U33.5
- new net ADDR33: R135.1, SJ34.2, U34.5
- new net ADDR34: R139.1, SJ35.2, U35.5
- new net ADDR35: R143.1, SJ36.2, U36.5
- new net ADDR36: R147.1, SJ37.2, U37.5
- new net ADDR37: R151.1, SJ38.2, U38.5
- new net ADDR38: R155.1, SJ39.2, U39.5
- new net ADDR39: R159.1, SJ40.2, U40.5
- new net ADDR4: R19.1, SJ5.2, U5.5
- new net ADDR40: R163.1, SJ41.2, U41.5
- new net ADDR41: R167.1, SJ42.2, U42.5
- new net ADDR42: R171.1, SJ43.2, U43.5
- new net ADDR43: R175.1, SJ44.2, U44.5
- new net ADDR44: R179.1, SJ45.2, U45.5
- new net ADDR45: R183.1, SJ46.2, U46.5
- new net ADDR46: R187.1, SJ47.2, U47.5
- new net ADDR47: R191.1, SJ48.2, U48.5
- new net ADDR48: R195.1, SJ49.2, U49.5
- new net ADDR49: R199.1, SJ50.2, U50.5
- new net ADDR5: R23.1, SJ6.2, U6.5
- new net ADDR6: R27.1, SJ7.2, U7.5
- new net ADDR7: R31.1, SJ8.2, U8.5
- new net ADDR8: R35.1, SJ9.2, U9.5
- new net ADDR9: R39.1, SJ10.2, U10.5
- new net GND1: C5.2, C7.2, C8.2, J5.1, J6.1, J7.1, R8.1, SJ2.1, U1.6
- new net GND10: C41.2, C43.2, C44.2, J41.1, J42.1, J43.1, R44.1, SJ11.1, U11.6
- new net GND11: C45.2, C47.2, C48.2, J45.1, J46.1, J47.1, R48.1, SJ12.1, U12.6
- new net GND12: C49.2, C51.2, C52.2, J49.1, J50.1, J51.1, R52.1, SJ13.1, U13.6
- new net GND13: C53.2, C55.2, C56.2, J53.1, J54.1, J55.1, R56.1, SJ14.1, U14.6
- new net GND14: C57.2, C59.2, C60.2, J57.1, J58.1, J59.1, R60.1, SJ15.1, U15.6
- new net GND15: C61.2, C63.2, C64.2, J61.1, J62.1, J63.1, R64.1, SJ16.1, U16.6
- new net GND16: C65.2, C67.2, C68.2, J65.1, J66.1, J67.1, R68.1, SJ17.1, U17.6
- new net GND17: C69.2, C71.2, C72.2, J69.1, J70.1, J71.1, R72.1, SJ18.1, U18.6
- new net GND18: C73.2, C75.2, C76.2, J73.1, J74.1, J75.1, R76.1, SJ19.1, U19.6
- new net GND19: C77.2, C79.2, C80.2, J77.1, J78.1, J79.1, R80.1, SJ20.1, U20.6
- new net GND2: C11.2, C12.2, C9.2, J10.1, J11.1, J9.1, R12.1, SJ3.1, U3.6
- new net GND20: C81.2, C83.2, C84.2, J81.1, J82.1, J83.1, R84.1, SJ21.1, U21.6
- new net GND21: C85.2, C87.2, C88.2, J85.1, J86.1, J87.1, R88.1, SJ22.1, U22.6
- new net GND22: C89.2, C91.2, C92.2, J89.1, J90.1, J91.1, R92.1, SJ23.1, U23.6
- new net GND23: C93.2, C95.2, C96.2, J93.1, J94.1, J95.1, R96.1, SJ24.1, U24.6
- new net GND24: C100.2, C97.2, C99.2, J97.1, J98.1, J99.1, R100.1, SJ25.1, U25.6
- new net GND25: C101.2, C103.2, C104.2, J101.1, J102.1, J103.1, R104.1, SJ26.1, U26.6
- new net GND26: C105.2, C107.2, C108.2, J105.1, J106.1, J107.1, R108.1, SJ27.1, U27.6
- new net GND27: C109.2, C111.2, C112.2, J109.1, J110.1, J111.1, R112.1, SJ28.1, U28.6
- new net GND28: C113.2, C115.2, C116.2, J113.1, J114.1, J115.1, R116.1, SJ29.1, U29.6
- new net GND29: C117.2, C119.2, C120.2, J117.1, J118.1, J119.1, R120.1, SJ30.1, U30.6
- new net GND3: C13.2, C15.2, C16.2, J13.1, J14.1, J15.1, R16.1, SJ4.1, U4.6
- new net GND30: C121.2, C123.2, C124.2, J121.1, J122.1, J123.1, R124.1, SJ31.1, U31.6
- new net GND31: C125.2, C127.2, C128.2, J125.1, J126.1, J127.1, R128.1, SJ32.1, U32.6
- new net GND32: C129.2, C131.2, C132.2, J129.1, J130.1, J131.1, R132.1, SJ33.1, U33.6
- new net GND33: C133.2, C135.2, C136.2, J133.1, J134.1, J135.1, R136.1, SJ34.1, U34.6
- new net GND34: C137.2, C139.2, C140.2, J137.1, J138.1, J139.1, R140.1, SJ35.1, U35.6
- new net GND35: C141.2, C143.2, C144.2, J141.1, J142.1, J143.1, R144.1, SJ36.1, U36.6
- new net GND36: C145.2, C147.2, C148.2, J145.1, J146.1, J147.1, R148.1, SJ37.1, U37.6
- new net GND37: C149.2, C151.2, C152.2, J149.1, J150.1, J151.1, R152.1, SJ38.1, U38.6
- new net GND38: C153.2, C155.2, C156.2, J153.1, J154.1, J155.1, R156.1, SJ39.1, U39.6
- new net GND39: C157.2, C159.2, C160.2, J157.1, J158.1, J159.1, R160.1, SJ40.1, U40.6
- new net GND4: C17.2, C19.2, C20.2, J17.1, J18.1, J19.1, R20.1, SJ5.1, U5.6
- new net GND40: C161.2, C163.2, C164.2, J161.1, J162.1, J163.1, R164.1, SJ41.1, U41.6
- new net GND41: C165.2, C167.2, C168.2, J165.1, J166.1, J167.1, R168.1, SJ42.1, U42.6
- new net GND42: C169.2, C171.2, C172.2, J169.1, J170.1, J171.1, R172.1, SJ43.1, U43.6
- new net GND43: C173.2, C175.2, C176.2, J173.1, J174.1, J175.1, R176.1, SJ44.1, U44.6
- new net GND44: C177.2, C179.2, C180.2, J177.1, J178.1, J179.1, R180.1, SJ45.1, U45.6
- new net GND45: C181.2, C183.2, C184.2, J181.1, J182.1, J183.1, R184.1, SJ46.1, U46.6
- new net GND46: C185.2, C187.2, C188.2, J185.1, J186.1, J187.1, R188.1, SJ47.1, U47.6
- new net GND47: C189.2, C191.2, C192.2, J189.1, J190.1, J191.1, R192.1, SJ48.1, U48.6
- new net GND48: C193.2, C195.2, C196.2, J193.1, J194.1, J195.1, R196.1, SJ49.1, U49.6
- new net GND49: C197.2, C199.2, C200.2, J197.1, J198.1, J199.1, R200.1, SJ50.1, U50.6
- new net GND5: C21.2, C23.2, C24.2, J21.1, J22.1, J23.1, R24.1, SJ6.1, U6.6
- new net GND6: C25.2, C27.2, C28.2, J25.1, J26.1, J27.1, R28.1, SJ7.1, U7.6
- new net GND7: C29.2, C31.2, C32.2, J29.1, J30.1, J31.1, R32.1, SJ8.1, U8.6
- new net GND8: C33.2, C35.2, C36.2, J33.1, J34.1, J35.1, R36.1, SJ9.1, U9.6
- new net GND9: C37.2, C39.2, C40.2, J37.1, J38.1, J39.1, R40.1, SJ10.1, U10.6
- new net INT1: J8.1, U1.4
- new net INT10: J44.1, U11.4
- new net INT11: J48.1, U12.4
- new net INT12: J52.1, U13.4
- new net INT13: J56.1, U14.4
- new net INT14: J60.1, U15.4
- new net INT15: J64.1, U16.4
- new net INT16: J68.1, U17.4
- new net INT17: J72.1, U18.4
- new net INT18: J76.1, U19.4
- new net INT19: J80.1, U20.4
- new net INT2: J12.1, U3.4
- new net INT20: J84.1, U21.4
- new net INT21: J88.1, U22.4
- new net INT22: J92.1, U23.4
- new net INT23: J96.1, U24.4
- new net INT24: J100.1, U25.4
- new net INT25: J104.1, U26.4
- new net INT26: J108.1, U27.4
- new net INT27: J112.1, U28.4
- new net INT28: J116.1, U29.4
- new net INT29: J120.1, U30.4
- new net INT3: J16.1, U4.4
- new net INT30: J124.1, U31.4
- new net INT31: J128.1, U32.4
- new net INT32: J132.1, U33.4
- new net INT33: J136.1, U34.4
- new net INT34: J140.1, U35.4
- new net INT35: J144.1, U36.4
- new net INT36: J148.1, U37.4
- new net INT37: J152.1, U38.4
- new net INT38: J156.1, U39.4
- new net INT39: J160.1, U40.4
- new net INT4: J20.1, U5.4
- new net INT40: J164.1, U41.4
- new net INT41: J168.1, U42.4
- new net INT42: J172.1, U43.4
- new net INT43: J176.1, U44.4
- new net INT44: J180.1, U45.4
- new net INT45: J184.1, U46.4
- new net INT46: J188.1, U47.4
- new net INT47: J192.1, U48.4
- new net INT48: J196.1, U49.4
- new net INT49: J200.1, U50.4
- new net INT5: J24.1, U6.4
- new net INT6: J28.1, U7.4
- new net INT7: J32.1, U8.4
- new net INT8: J36.1, U9.4
- new net INT9: J40.1, U10.4
- new net N$10: C6.2, R8.2
- new net N$100: C78.2, R80.2
- new net N$101: JP145.1, R82.2
- new net N$102: JP145.3, R81.2
- new net N$103: C83.1, U21.12
- new net N$104: C82.1, U21.10
- new net N$105: C82.2, R84.2
- new net N$106: JP152.1, R86.2
- new net N$107: JP152.3, R85.2
- new net N$108: C87.1, U22.12
- new net N$109: C86.1, U22.10
- new net N$11: JP19.1, R10.2
- new net N$110: C86.2, R88.2
- new net N$111: JP159.1, R90.2
- new net N$112: JP159.3, R89.2
- new net N$113: C91.1, U23.12
- new net N$114: C90.1, U23.10
- new net N$115: C90.2, R92.2
- new net N$116: JP166.1, R94.2
- new net N$117: JP166.3, R93.2
- new net N$118: C95.1, U24.12
- new net N$119: C94.1, U24.10
- new net N$12: JP19.3, R9.2
- new net N$120: C94.2, R96.2
- new net N$121: JP173.1, R98.2
- new net N$122: JP173.3, R97.2
- new net N$123: C99.1, U25.12
- new net N$124: C98.1, U25.10
- new net N$125: C98.2, R100.2
- new net N$126: JP180.1, R102.2
- new net N$127: JP180.3, R101.2
- new net N$128: C103.1, U26.12
- new net N$129: C102.1, U26.10
- new net N$13: C11.1, U3.12
- new net N$130: C102.2, R104.2
- new net N$131: JP187.1, R106.2
- new net N$132: JP187.3, R105.2
- new net N$133: C107.1, U27.12
- new net N$134: C106.1, U27.10
- new net N$135: C106.2, R108.2
- new net N$136: JP194.1, R110.2
- new net N$137: JP194.3, R109.2
- new net N$138: C111.1, U28.12
- new net N$139: C110.1, U28.10
- new net N$14: C10.1, U3.10
- new net N$140: C110.2, R112.2
- new net N$141: JP201.1, R114.2
- new net N$142: JP201.3, R113.2
- new net N$143: C115.1, U29.12
- new net N$144: C114.1, U29.10
- new net N$145: C114.2, R116.2
- new net N$146: JP208.1, R118.2
- new net N$147: JP208.3, R117.2
- new net N$148: C119.1, U30.12
- new net N$149: C118.1, U30.10
- new net N$15: C10.2, R12.2
- new net N$150: C118.2, R120.2
- new net N$151: JP215.1, R122.2
- new net N$152: JP215.3, R121.2
- new net N$153: C123.1, U31.12
- new net N$154: C122.1, U31.10
- new net N$155: C122.2, R124.2
- new net N$156: JP222.1, R126.2
- new net N$157: JP222.3, R125.2
- new net N$158: C127.1, U32.12
- new net N$159: C126.1, U32.10
- new net N$16: JP26.1, R14.2
- new net N$160: C126.2, R128.2
- new net N$161: JP229.1, R130.2
- new net N$162: JP229.3, R129.2
- new net N$163: C131.1, U33.12
- new net N$164: C130.1, U33.10
- new net N$165: C130.2, R132.2
- new net N$166: JP236.1, R134.2
- new net N$167: JP236.3, R133.2
- new net N$168: C135.1, U34.12
- new net N$169: C134.1, U34.10
- new net N$17: JP26.3, R13.2
- new net N$170: C134.2, R136.2
- new net N$171: JP243.1, R138.2
- new net N$172: JP243.3, R137.2
- new net N$173: C139.1, U35.12
- new net N$174: C138.1, U35.10
- new net N$175: C138.2, R140.2
- new net N$176: JP250.1, R142.2
- new net N$177: JP250.3, R141.2
- new net N$178: C143.1, U36.12
- new net N$179: C142.1, U36.10
- new net N$18: C15.1, U4.12
- new net N$180: C142.2, R144.2
- new net N$181: JP257.1, R146.2
- new net N$182: JP257.3, R145.2
- new net N$183: C147.1, U37.12
- new net N$184: C146.1, U37.10
- new net N$185: C146.2, R148.2
- new net N$186: JP264.1, R150.2
- new net N$187: JP264.3, R149.2
- new net N$188: C151.1, U38.12
- new net N$189: C150.1, U38.10
- new net N$19: C14.1, U4.10
- new net N$190: C150.2, R152.2
- new net N$191: JP271.1, R154.2
- new net N$192: JP271.3, R153.2
- new net N$193: C155.1, U39.12
- new net N$194: C154.1, U39.10
- new net N$195: C154.2, R156.2
- new net N$196: JP278.1, R158.2
- new net N$197: JP278.3, R157.2
- new net N$198: C159.1, U40.12
- new net N$199: C158.1, U40.10
- new net N$20: C14.2, R16.2
- new net N$200: C158.2, R160.2
- new net N$201: JP285.1, R162.2
- new net N$202: JP285.3, R161.2
- new net N$203: C163.1, U41.12
- new net N$204: C162.1, U41.10
- new net N$205: C162.2, R164.2
- new net N$206: JP292.1, R166.2
- new net N$207: JP292.3, R165.2
- new net N$208: C167.1, U42.12
- new net N$209: C166.1, U42.10
- new net N$21: JP33.1, R18.2
- new net N$210: C166.2, R168.2
- new net N$211: JP299.1, R170.2
- new net N$212: JP299.3, R169.2
- new net N$213: C171.1, U43.12
- new net N$214: C170.1, U43.10
- new net N$215: C170.2, R172.2
- new net N$216: JP306.1, R174.2
- new net N$217: JP306.3, R173.2
- new net N$218: C175.1, U44.12
- new net N$219: C174.1, U44.10
- new net N$22: JP33.3, R17.2
- new net N$220: C174.2, R176.2
- new net N$221: JP313.1, R178.2
- new net N$222: JP313.3, R177.2
- new net N$223: C179.1, U45.12
- new net N$224: C178.1, U45.10
- new net N$225: C178.2, R180.2
- new net N$226: JP320.1, R182.2
- new net N$227: JP320.3, R181.2
- new net N$228: C183.1, U46.12
- new net N$229: C182.1, U46.10
- new net N$23: C19.1, U5.12
- new net N$230: C182.2, R184.2
- new net N$231: JP327.1, R186.2
- new net N$232: JP327.3, R185.2
- new net N$233: C187.1, U47.12
- new net N$234: C186.1, U47.10
- new net N$235: C186.2, R188.2
- new net N$236: JP334.1, R190.2
- new net N$237: JP334.3, R189.2
- new net N$238: C191.1, U48.12
- new net N$239: C190.1, U48.10
- new net N$24: C18.1, U5.10
- new net N$240: C190.2, R192.2
- new net N$241: JP341.1, R194.2
- new net N$242: JP341.3, R193.2
- new net N$243: C195.1, U49.12
- new net N$244: C194.1, U49.10
- new net N$245: C194.2, R196.2
- new net N$246: JP348.1, R198.2
- new net N$247: JP348.3, R197.2
- new net N$248: C199.1, U50.12
- new net N$249: C198.1, U50.10
- new net N$25: C18.2, R20.2
- new net N$250: C198.2, R200.2
- new net N$26: JP40.1, R22.2
- new net N$27: JP40.3, R21.2
- new net N$28: C23.1, U6.12
- new net N$29: C22.1, U6.10
- new net N$30: C22.2, R24.2
- new net N$31: JP47.1, R26.2
- new net N$32: JP47.3, R25.2
- new net N$33: C27.1, U7.12
- new net N$34: C26.1, U7.10
- new net N$35: C26.2, R28.2
- new net N$36: JP54.1, R30.2
- new net N$37: JP54.3, R29.2
- new net N$38: C31.1, U8.12
- new net N$39: C30.1, U8.10
- new net N$40: C30.2, R32.2
- new net N$41: JP61.1, R34.2
- new net N$42: JP61.3, R33.2
- new net N$43: C35.1, U9.12
- new net N$44: C34.1, U9.10
- new net N$45: C34.2, R36.2
- new net N$46: JP68.1, R38.2
- new net N$47: JP68.3, R37.2
- new net N$48: C39.1, U10.12
- new net N$49: C38.1, U10.10
- new net N$50: C38.2, R40.2
- new net N$51: JP75.1, R42.2
- new net N$52: JP75.3, R41.2
- new net N$53: C43.1, U11.12
- new net N$54: C42.1, U11.10
- new net N$55: C42.2, R44.2
- new net N$56: JP82.1, R46.2
- new net N$57: JP82.3, R45.2
- new net N$58: C47.1, U12.12
- new net N$59: C46.1, U12.10
- new net N$6: JP12.1, R6.2
- new net N$60: C46.2, R48.2
- new net N$61: JP89.1, R50.2
- new net N$62: JP89.3, R49.2
- new net N$63: C51.1, U13.12
- new net N$64: C50.1, U13.10
- new net N$65: C50.2, R52.2
- new net N$66: JP96.1, R54.2
- new net N$67: JP96.3, R53.2
- new net N$68: C55.1, U14.12
- new net N$69: C54.1, U14.10
- new net N$7: JP12.3, R3.2
- new net N$70: C54.2, R56.2
- new net N$71: JP103.1, R58.2
- new net N$72: JP103.3, R57.2
- new net N$73: C59.1, U15.12
- new net N$74: C58.1, U15.10
- new net N$75: C58.2, R60.2
- new net N$76: JP110.1, R62.2
- new net N$77: JP110.3, R61.2
- new net N$78: C63.1, U16.12
- new net N$79: C62.1, U16.10
- new net N$8: C7.1, U1.12
- new net N$80: C62.2, R64.2
- new net N$81: JP117.1, R66.2
- new net N$82: JP117.3, R65.2
- new net N$83: C67.1, U17.12
- new net N$84: C66.1, U17.10
- new net N$85: C66.2, R68.2
- new net N$86: JP124.1, R70.2
- new net N$87: JP124.3, R69.2
- new net N$88: C71.1, U18.12
- new net N$89: C70.1, U18.10
- new net N$9: C6.1, U1.10
- new net N$90: C70.2, R72.2
- new net N$91: JP131.1, R74.2
- new net N$92: JP131.3, R73.2
- new net N$93: C75.1, U19.12
- new net N$94: C74.1, U19.10
- new net N$95: C74.2, R76.2
- new net N$96: JP138.1, R78.2
- new net N$97: JP138.3, R77.2
- new net N$98: C79.1, U20.12
- new net N$99: C78.1, U20.10
- new net SCL1: J5.4, J6.4, J7.4, R3.1, U1.3
- new net SCL10: J41.4, J42.4, J43.4, R41.1, U11.3
- new net SCL11: J45.4, J46.4, J47.4, R45.1, U12.3
- new net SCL12: J49.4, J50.4, J51.4, R49.1, U13.3
- new net SCL13: J53.4, J54.4, J55.4, R53.1, U14.3
- new net SCL14: J57.4, J58.4, J59.4, R57.1, U15.3
- new net SCL15: J61.4, J62.4, J63.4, R61.1, U16.3
- new net SCL16: J65.4, J66.4, J67.4, R65.1, U17.3
- new net SCL17: J69.4, J70.4, J71.4, R69.1, U18.3
- new net SCL18: J73.4, J74.4, J75.4, R73.1, U19.3
- new net SCL19: J77.4, J78.4, J79.4, R77.1, U20.3
- new net SCL2: J10.4, J11.4, J9.4, R9.1, U3.3
- new net SCL20: J81.4, J82.4, J83.4, R81.1, U21.3
- new net SCL21: J85.4, J86.4, J87.4, R85.1, U22.3
- new net SCL22: J89.4, J90.4, J91.4, R89.1, U23.3
- new net SCL23: J93.4, J94.4, J95.4, R93.1, U24.3
- new net SCL24: J97.4, J98.4, J99.4, R97.1, U25.3
- new net SCL25: J101.4, J102.4, J103.4, R101.1, U26.3
- new net SCL26: J105.4, J106.4, J107.4, R105.1, U27.3
- new net SCL27: J109.4, J110.4, J111.4, R109.1, U28.3
- new net SCL28: J113.4, J114.4, J115.4, R113.1, U29.3
- new net SCL29: J117.4, J118.4, J119.4, R117.1, U30.3
- new net SCL3: J13.4, J14.4, J15.4, R13.1, U4.3
- new net SCL30: J121.4, J122.4, J123.4, R121.1, U31.3
- new net SCL31: J125.4, J126.4, J127.4, R125.1, U32.3
- new net SCL32: J129.4, J130.4, J131.4, R129.1, U33.3
- new net SCL33: J133.4, J134.4, J135.4, R133.1, U34.3
- new net SCL34: J137.4, J138.4, J139.4, R137.1, U35.3
- new net SCL35: J141.4, J142.4, J143.4, R141.1, U36.3
- new net SCL36: J145.4, J146.4, J147.4, R145.1, U37.3
- new net SCL37: J149.4, J150.4, J151.4, R149.1, U38.3
- new net SCL38: J153.4, J154.4, J155.4, R153.1, U39.3
- new net SCL39: J157.4, J158.4, J159.4, R157.1, U40.3
- new net SCL4: J17.4, J18.4, J19.4, R17.1, U5.3
- new net SCL40: J161.4, J162.4, J163.4, R161.1, U41.3
- new net SCL41: J165.4, J166.4, J167.4, R165.1, U42.3
- new net SCL42: J169.4, J170.4, J171.4, R169.1, U43.3
- new net SCL43: J173.4, J174.4, J175.4, R173.1, U44.3
- new net SCL44: J177.4, J178.4, J179.4, R177.1, U45.3
- new net SCL45: J181.4, J182.4, J183.4, R181.1, U46.3
- new net SCL46: J185.4, J186.4, J187.4, R185.1, U47.3
- new net SCL47: J189.4, J190.4, J191.4, R189.1, U48.3
- new net SCL48: J193.4, J194.4, J195.4, R193.1, U49.3
- new net SCL49: J197.4, J198.4, J199.4, R197.1, U50.3
- new net SCL5: J21.4, J22.4, J23.4, R21.1, U6.3
- new net SCL6: J25.4, J26.4, J27.4, R25.1, U7.3
- new net SCL7: J29.4, J30.4, J31.4, R29.1, U8.3
- new net SCL8: J33.4, J34.4, J35.4, R33.1, U9.3
- new net SCL9: J37.4, J38.4, J39.4, R37.1, U10.3
- new net SDA1: J5.3, J6.3, J7.3, R6.1, U1.2
- new net SDA10: J41.3, J42.3, J43.3, R42.1, U11.2
- new net SDA11: J45.3, J46.3, J47.3, R46.1, U12.2
- new net SDA12: J49.3, J50.3, J51.3, R50.1, U13.2
- new net SDA13: J53.3, J54.3, J55.3, R54.1, U14.2
- new net SDA14: J57.3, J58.3, J59.3, R58.1, U15.2
- new net SDA15: J61.3, J62.3, J63.3, R62.1, U16.2
- new net SDA16: J65.3, J66.3, J67.3, R66.1, U17.2
- new net SDA17: J69.3, J70.3, J71.3, R70.1, U18.2
- new net SDA18: J73.3, J74.3, J75.3, R74.1, U19.2
- new net SDA19: J77.3, J78.3, J79.3, R78.1, U20.2
- new net SDA2: J10.3, J11.3, J9.3, R10.1, U3.2
- new net SDA20: J81.3, J82.3, J83.3, R82.1, U21.2
- new net SDA21: J85.3, J86.3, J87.3, R86.1, U22.2
- new net SDA22: J89.3, J90.3, J91.3, R90.1, U23.2
- new net SDA23: J93.3, J94.3, J95.3, R94.1, U24.2
- new net SDA24: J97.3, J98.3, J99.3, R98.1, U25.2
- new net SDA25: J101.3, J102.3, J103.3, R102.1, U26.2
- new net SDA26: J105.3, J106.3, J107.3, R106.1, U27.2
- new net SDA27: J109.3, J110.3, J111.3, R110.1, U28.2
- new net SDA28: J113.3, J114.3, J115.3, R114.1, U29.2
- new net SDA29: J117.3, J118.3, J119.3, R118.1, U30.2
- new net SDA3: J13.3, J14.3, J15.3, R14.1, U4.2
- new net SDA30: J121.3, J122.3, J123.3, R122.1, U31.2
- new net SDA31: J125.3, J126.3, J127.3, R126.1, U32.2
- new net SDA32: J129.3, J130.3, J131.3, R130.1, U33.2
- new net SDA33: J133.3, J134.3, J135.3, R134.1, U34.2
- new net SDA34: J137.3, J138.3, J139.3, R138.1, U35.2
- new net SDA35: J141.3, J142.3, J143.3, R142.1, U36.2
- new net SDA36: J145.3, J146.3, J147.3, R146.1, U37.2
- new net SDA37: J149.3, J150.3, J151.3, R150.1, U38.2
- new net SDA38: J153.3, J154.3, J155.3, R154.1, U39.2
- new net SDA39: J157.3, J158.3, J159.3, R158.1, U40.2
- new net SDA4: J17.3, J18.3, J19.3, R18.1, U5.2
- new net SDA40: J161.3, J162.3, J163.3, R162.1, U41.2
- new net SDA41: J165.3, J166.3, J167.3, R166.1, U42.2
- new net SDA42: J169.3, J170.3, J171.3, R170.1, U43.2
- new net SDA43: J173.3, J174.3, J175.3, R174.1, U44.2
- new net SDA44: J177.3, J178.3, J179.3, R178.1, U45.2
- new net SDA45: J181.3, J182.3, J183.3, R182.1, U46.2
- new net SDA46: J185.3, J186.3, J187.3, R186.1, U47.2
- new net SDA47: J189.3, J190.3, J191.3, R190.1, U48.2
- new net SDA48: J193.3, J194.3, J195.3, R194.1, U49.2
- new net SDA49: J197.3, J198.3, J199.3, R198.1, U50.2
- new net SDA5: J21.3, J22.3, J23.3, R22.1, U6.2
- new net SDA6: J25.3, J26.3, J27.3, R26.1, U7.2
- new net SDA7: J29.3, J30.3, J31.3, R30.1, U8.2
- new net SDA8: J33.3, J34.3, J35.3, R34.1, U9.2
- new net SDA9: J37.3, J38.3, J39.3, R38.1, U10.2
Routing:
- net SCL45: track 0.00 -> 59.2 mm, vias 0 -> 2
- net SCL34: track 0.00 -> 59.2 mm, vias 0 -> 2
- net SCL24: track 0.00 -> 59.2 mm, vias 0 -> 2
- net SCL11: track 0.00 -> 59.2 mm, vias 0 -> 2
- net SCL5: track 0.00 -> 59.2 mm, vias 0 -> 2
- net SCL40: track 0.00 -> 59.2 mm, vias 0 -> 2
- net SCL4: track 0.00 -> 59.2 mm, vias 0 -> 2
- net SCL35: track 0.00 -> 59.2 mm, vias 0 -> 2
- net SCL25: track 0.00 -> 59.2 mm, vias 0 -> 2
- net SCL15: track 0.00 -> 59.2 mm, vias 0 -> 2
- net SCL10: track 0.00 -> 59.2 mm, vias 0 -> 2
- net SCL1: track 0.00 -> 59.2 mm, vias 0 -> 2
- net SCL44: track 0.00 -> 59.2 mm, vias 0 -> 2
- net SCL41: track 0.00 -> 59.2 mm, vias 0 -> 2
- net SCL31: track 0.00 -> 59.2 mm, vias 0 -> 2
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- added copper zone on layer 1, net GND1
- added copper zone on layer 16, net GND1
- added copper zone on layer 1, net GND10
- added copper zone on layer 16, net GND10
- added copper zone on layer 1, net GND11
- added copper zone on layer 16, net GND11
- added copper zone on layer 1, net GND12
- added copper zone on layer 16, net GND12
- added copper zone on layer 1, net GND13
- added copper zone on layer 16, net GND13
- added copper zone on layer 1, net GND14
- added copper zone on layer 16, net GND14
- added copper zone on layer 1, net GND15
- added copper zone on layer 16, net GND15
- added copper zone on layer 1, net GND16
- added copper zone on layer 16, net GND16
- added copper zone on layer 1, net GND17
- added copper zone on layer 16, net GND17
- added copper zone on layer 1, net GND18
- added copper zone on layer 16, net GND18
- added copper zone on layer 1, net GND19
- added copper zone on layer 16, net GND19
- added copper zone on layer 1, net GND2
- added copper zone on layer 16, net GND2
- added copper zone on layer 1, net GND20
- added copper zone on layer 16, net GND20
- added copper zone on layer 1, net GND21
- added copper zone on layer 16, net GND21
- added copper zone on layer 1, net GND22
- added copper zone on layer 16, net GND22
- added copper zone on layer 1, net GND23
- added copper zone on layer 16, net GND23
- added copper zone on layer 1, net GND24
- added copper zone on layer 16, net GND24
- added copper zone on layer 1, net GND25
- added copper zone on layer 16, net GND25
- added copper zone on layer 1, net GND26
- added copper zone on layer 16, net GND26
- added copper zone on layer 1, net GND27
- added copper zone on layer 16, net GND27
- added copper zone on layer 1, net GND28
- added copper zone on layer 16, net GND28
- added copper zone on layer 1, net GND29
- added copper zone on layer 16, net GND29
- added copper zone on layer 1, net GND3
- added copper zone on layer 16, net GND3
- added copper zone on layer 1, net GND30
- added copper zone on layer 16, net GND30
- added copper zone on layer 1, net GND31
- added copper zone on layer 16, net GND31
- added copper zone on layer 1, net GND32
- added copper zone on layer 16, net GND32
- added copper zone on layer 1, net GND33
- added copper zone on layer 16, net GND33
- added copper zone on layer 1, net GND34
- added copper zone on layer 16, net GND34
- added copper zone on layer 1, net GND35
- added copper zone on layer 16, net GND35
- added copper zone on layer 1, net GND36
- added copper zone on layer 16, net GND36
- added copper zone on layer 1, net GND37
- added copper zone on layer 16, net GND37
- added copper zone on layer 1, net GND38
- added copper zone on layer 16, net GND38
- added copper zone on layer 1, net GND39
- added copper zone on layer 16, net GND39
- added copper zone on layer 1, net GND4
- added copper zone on layer 16, net GND4
- added copper zone on layer 1, net GND40
- added copper zone on layer 16, net GND40
- added copper zone on layer 1, net GND41
- added copper zone on layer 16, net GND41
- added copper zone on layer 1, net GND42
- added copper zone on layer 16, net GND42
- added copper zone on layer 1, net GND43
- added copper zone on layer 16, net GND43
- added copper zone on layer 1, net GND44
- added copper zone on layer 16, net GND44
- added copper zone on layer 1, net GND45
- added copper zone on layer 16, net GND45
- added copper zone on layer 1, net GND46
- added copper zone on layer 16, net GND46
- added copper zone on layer 1, net GND47
- added copper zone on layer 16, net GND47
- added copper zone on layer 1, net GND48
- added copper zone on layer 16, net GND48
- added copper zone on layer 1, net GND49
- added copper zone on layer 16, net GND49
- added copper zone on layer 1, net GND5
- added copper zone on layer 16, net GND5
- added copper zone on layer 1, net GND6
- added copper zone on layer 16, net GND6
- added copper zone on layer 1, net GND7
- added copper zone on layer 16, net GND7
- added copper zone on layer 1, net GND8
- added copper zone on layer 16, net GND8
- added copper zone on layer 1, net GND9
- added copper zone on layer 16, net GND9
Other:
- board size 25.4 x 25.4 mm -> 272.3 x 142.7 mm
